Commit message: error fixed on ros2_control xacro

File: description/ros2_control.xacro (robot description, xacro)
@@ -1,4 +1,5 @@
 <?xml version="1.0"?>
 <robot xmlns:xacro="http://www.ros.org/wiki/xacro" >
+    <xacro:macro name="ros2_control" params="">
       <ros2_control name="RealRobot" type="system">
             <hardware>
@@ -29,3 +30,4 @@
             </joint>
         </ros2_control>
+       </xacro:macro>
 </robot>
