Commit message: 5 commit

File: description/complete.xacro (robot description, xacro)
@@ -2,3 +2,4 @@
 <robot xmlns:xacro="http://www.ros.org/wiki/xacro" name="eve_bot">
   <xacro:include filename="robot.urdf.xacro" />
+  <xacro:include filename="lidar.xacro" />
 </robot>

File: description/lidar.xacro (robot description, xacro)
@@ -1,4 +1,5 @@
 <?xml version="1.0"?>
 <robot xmlns:xacro="http://www.ros.org/wiki/xacro" >
+    <xacro:include filename="inertial_macros.xacro" />
     <material name="red">
      <color rgba="1 0 0 1"/>
@@ -7,5 +8,5 @@
      <visual>
          <geometry>
-           <cylinder radius="0.035" length="0.035"/>
+           <cylinder radius="0.035" length="0.0545"/>
          </geometry>
          <origin xyz="0 0 0" rpy="0 0 0"/>
@@ -14,14 +15,14 @@
      <collision>
           <geometry>
-           <cylinder radius="0.035" length="0.035"/>
+           <cylinder radius="0.035" length="0.0545"/>
          </geometry>
          <origin xyz="0 0 0" rpy="0 0 0"/>
      </collision>
-     <xacro:cylinder_inertia m="0.3" r="0.035" l="0.035" o_xyz="0 0 0" o_rpy="0 0 0" />
+     <xacro:cylinder_inertia m="0.3" r="0.035" l="0.0545" o_xyz="0 0 0" o_rpy="0 0 0" />
     </link>
     <joint name="laser_joint" type="fixed">
         <parent link="base_link"/>
         <child link="lidar_frame"/>
-        <origin xyz="0.065 0 0.0795" rpy="0 0 3.14"/>
+        <origin xyz="0 0 0.06225" rpy="0 0 0"/>
     </joint>
     <!--<gazebo reference="lidar_frame">

File: description/robot.urdf.xacro (robot description, xacro)
@@ -31,5 +31,5 @@
        <parent link="base_footprint"/>
        <child link="base_link"/>
-       <origin xyz="0 0 0.035" rpy="0 0 0"/>
+       <origin xyz="0 0 0.042" rpy="0 0 0"/>
    </joint>
    <link name="raspberry_link">
@@ -52,5 +52,5 @@
       <parent link="base_link"/>
       <child link="raspberry_link"/>
-      <origin xyz="-0.10 0 0.07" rpy="0 0 0"/>
+      <origin xyz="-0.10 0 0.0525" rpy="0 0 0"/>
    </joint>
    <link name="right_wheel_link">
@@ -73,5 +73,5 @@
       <parent link="base_link"/>
       <child link="right_wheel_link"/>
-      <origin xyz="0 -0.115 0" rpy="0 0 0"/>
+      <origin xyz="0 -0.115 -0.009" rpy="0 0 0"/>
       <axis xyz="0 1 0"/>
    </joint>
@@ -95,5 +95,5 @@
       <parent link="base_link"/>
       <child link="left_wheel_link"/>
-      <origin xyz="0 0.115 0" rpy="0 0 0"/>
+      <origin xyz="0 0.115 -0.009" rpy="0 0 0"/>
       <axis xyz="0 1 0"/>
    </joint>
@@ -101,5 +101,5 @@
       <visual>
          <geometry>
-           <sphere radius="0.017"/>
+           <sphere radius="0.033"/>
          </geometry>
          <origin xyz="0 0 0" rpy="0 0 0"/>
@@ -108,14 +108,14 @@
       <collision>
          <geometry>
-           <sphere radius="0.017"/>
+           <sphere radius="0.033"/>
          </geometry>
          <origin xyz="0 0 0" rpy="0 0 0"/>
       </collision>
-      <xacro:sphere_inertia m="0.2" r="0.017" o_xyz="0 0 0" o_rpy="0 0 0" />
+      <xacro:sphere_inertia m="0.2" r="0.033" o_xyz="0 0 0" o_rpy="0 0 0" />
    </link>
    <joint name="base_caster_wheel_joint" type="fixed">
        <parent link="base_link"/>
        <child link="caster_wheel_link"/>
-       <origin xyz="0.085 0 -0.062" rpy="0 0 0"/>
+       <origin xyz="0.12 0 -0.009" rpy="0 0 0"/>
    </joint>
 </robot>

Commit message: error fixed on ros2_control xacro

File: description/complete.xacro (robot description, xacro)
@@ -2,4 +2,5 @@
 <robot xmlns:xacro="http://www.ros.org/wiki/xacro" name="eve_bot">
   <xacro:arg name="use_ros2_control" default="true" />
+  <xacro:arg name="sim_mode" default="false" />
   <xacro:include filename="ros2_control.xacro" />
   <xacro:include filename="robot.urdf.xacro" />

File: description/lidar.xacro (robot description, xacro)
@@ -1,4 +1,7 @@
 <?xml version="1.0"?>
 <robot xmlns:xacro="http://www.ros.org/wiki/xacro" >
+    <material name="black">
+     <color rgba="0 0 0 1"/>
+   </material>
     <joint name="laser_joint" type="fixed">
         <parent link="base_link"/>

Commit message: error fixed on ros2_control xacro

File: description/complete.xacro (robot description, xacro)
@@ -3,6 +3,6 @@
   <xacro:arg name="use_ros2_control" default="true" />
   <xacro:arg name="sim_mode" default="false" />
+  <xacro:include filename="robot.urdf.xacro" />
   <xacro:include filename="ros2_control.xacro" />
-  <xacro:include filename="robot.urdf.xacro" />
   <xacro:include filename="lidar.xacro" />
 </robot>

File: description/ros2_control.xacro (robot description, xacro)
@@ -1,5 +1,4 @@
 <?xml version="1.0"?>
 <robot xmlns:xacro="http://www.ros.org/wiki/xacro" >
-    <xacro:macro name="ros2_control" params="">
       <ros2_control name="RealRobot" type="system">
             <hardware>
@@ -18,6 +17,6 @@
                     <param name="max">10</param>
                 </command_interface>
+                <state_interface name="position"/>
                 <state_interface name="velocity"/>
-                <state_interface name="position"/>
             </joint>
             <joint name="right_wheel_joint">
@@ -26,8 +25,7 @@
                     <param name="max">10</param>
                 </command_interface>
+                <state_interface name="position"/>
                 <state_interface name="velocity"/>
-                <state_interface name="position"/>
             </joint>
         </ros2_control>
-       </xacro:macro>
 </robot>

Commit message: error fixed on ros2_control xacro

File: description/complete.xacro (robot description, xacro)
@@ -1,5 +1,4 @@
 <?xml version="1.0"?>
 <robot xmlns:xacro="http://www.ros.org/wiki/xacro" name="eve_bot">
-  <xacro:arg name="use_ros2_control" default="true" />
   <xacro:arg name="sim_mode" default="false" />
   <xacro:include filename="robot.urdf.xacro" />

File: description/lidar.xacro (robot description, xacro)
@@ -5,5 +5,5 @@
    </material>
     <joint name="laser_joint" type="fixed">
-        <parent link="base_link"/>
+        <parent link="chassis"/>
         <child link="laser_frame"/>
         <origin xyz="0 0 0.06" rpy="0 0 0"/>

File: description/robot.urdf.xacro (robot description, xacro)
@@ -12,10 +12,4 @@
    </material>
    <link name="base_link"/>
-   <joint name="base_footprint_joint" type="fixed">
-       <parent link="base_link"/>
-       <child link="base_footprint"/>
-       <origin xyz="0 0 0" rpy="0 0 0"/>
-   </joint>
-   <link name="base_footprint"/>
    <link name="chassis">
       <visual>

Commit message: add camera

File: description/complete.xacro (robot description, xacro)
@@ -3,5 +3,7 @@
   <xacro:arg name="sim_mode" default="false" />
   <xacro:include filename="robot.urdf.xacro" />
+  <xacro:include filename="lidar.xacro" />
+  <xacro:include filename="upbody.xacro" />
   <xacro:include filename="ros2_control.xacro" />
-  <xacro:include filename="lidar.xacro" />
+  <xacro:include filename="camera.xacro" />
 </robot>

File: description/lidar.xacro (robot description, xacro)
@@ -7,13 +7,7 @@
         <parent link="chassis"/>
         <child link="laser_frame"/>
-        <origin xyz="0 0 0.115" rpy="0 0 0"/>
+        <origin xyz="0 0 0.095" rpy="0 0 0"/>
     </joint>
     <link name="laser_frame">
-        <visual>
-            <geometry>
-                <cylinder radius="0.034" length="0.05"/>
-            </geometry>
-            <material name="black"/>
-        </visual>
         <visual>
             <origin xyz="0 0 0"/>

File: description/robot.urdf.xacro (robot description, xacro)
@@ -2,106 +2,100 @@
 <robot name="robot" xmlns:xacro="http://www.ros.org/wiki/xacro">
   <xacro:include filename="inertial_macros.xacro" />
-   <material name="white">
-     <color rgba="1 1 1 1"/>
-   </material>
-   <material name="green">
-     <color rgba="0 1 0 1"/>
-   </material>
-   <material name="gray">
-     <color rgba="0.5 0.5 0.5 1"/>
-   </material>
-   <link name="base_link"/>
-   <joint name="base_footprint_joint" type="fixed">
-        <parent link="base_link"/>
-        <child link="base_footprint"/>
-        <origin xyz="0 0 0" rpy="0 0 0"/>
-    </joint>
-    <link name="base_footprint">
-    </link>
-   <link name="chassis">
-      <visual>
-        <geometry>
-          <cylinder radius="0.17" length="0.14"/>
-        </geometry>
-        <origin xyz="0 0 0" rpy="0 0 0"/>
-        <material name="white"/>
-      </visual>
-      <collision>
-        <geometry>
-          <cylinder radius="0.17" length="0.14"/>
-        </geometry>
-        <origin xyz="0 0 0" rpy="0 0 0"/>
-      </collision>
-      <xacro:cylinder_inertia m="4" r="0.17" l="0.14" o_xyz="0 0 0" o_rpy="0 0 0" />
-   </link>
-   <joint name="chassis_joint" type="fixed">
-       <parent link="base_link"/>
-       <child link="chassis"/>
-       <origin xyz="0 0 0.07" rpy="0 0 0"/>
-   </joint>
-   <link name="right_wheel">
-      <visual>
-         <geometry>
-           <cylinder radius="0.033" length="0.015"/>
-         </geometry>
-         <origin xyz="0 0 0" rpy="1.57 0 0"/>
-         <material name="gray"/>
-      </visual>
-      <collision>
-         <geometry>
-           <cylinder radius="0.033" length="0.015"/>
-         </geometry>
-         <origin xyz="0 0 0" rpy="1.57 0 0"/>
-      </collision>
-      <xacro:cylinder_inertia m="0.2" r="0.033" l="0.015" o_xyz="0 0 0" o_rpy="1.57 0 0" />
-   </link>
-   <joint name="right_wheel_joint" type="continuous">
-      <parent link="chassis"/>
-      <child link="right_wheel"/>
-      <origin xyz="0 -0.115 -0.017" rpy="0 0 0"/>
-      <axis xyz="0 1 0"/>
-   </joint>
-   <link name="left_wheel">
-      <visual>
-         <geometry>
-           <cylinder radius="0.033" length="0.015"/>
-         </geometry>
-         <origin xyz="0 0 0" rpy="1.57 0 0"/>
-         <material name="gray"/>
-      </visual>
-      <collision>
-         <geometry>
-           <cylinder radius="0.033" length="0.015"/>
-         </geometry>
-         <origin xyz="0 0 0" rpy="1.57 0 0"/>
-      </collision>
-      <xacro:cylinder_inertia m="0.2" r="0.033" l="0.015" o_xyz="0 0 0" o_rpy="1.57 0 0" />
-   </link>
-   <joint name="left_wheel_joint" type="continuous">
-      <parent link="chassis"/>
-      <child link="left_wheel"/>
-      <origin xyz="0 0.115 -0.017" rpy="0 0 0"/>
-      <axis xyz="0 1 0"/>
-   </joint>
-   <link name="caster_wheel">
-      <visual>
-         <geometry>
-           <sphere radius="0.033"/>
-         </geometry>
-         <origin xyz="0 0 0" rpy="0 0 0"/>
-         <material name="gray"/>
-      </visual>
-      <collision>
-         <geometry>
-           <sphere radius="0.033"/>
-         </geometry>
-         <origin xyz="0 0 0" rpy="0 0 0"/>
-      </collision>
-      <xacro:sphere_inertia m="0.2" r="0.033" o_xyz="0 0 0" o_rpy="0 0 0" />
-   </link>
-   <joint name="caster_wheel_joint" type="fixed">
-       <parent link="chassis"/>
-       <child link="caster_wheel"/>
-       <origin xyz="0.12 0 -0.017" rpy="0 0 0"/>
-   </joint>
+  <material name="white">
+   <color rgba="1 1 1 1"/>
+  </material>
+  <material name="green">
+   <color rgba="0 1 0 1"/>
+  </material>
+  <material name="gray">
+   <color rgba="0.5 0.5 0.5 1"/>
+  </material>
+ <link name="base_footprint"/>
+ <!-- Chassis link -->
+ <joint name="chassis_joint" type="fixed">
+   <parent link="base_footprint"/>
+   <child link="chassis"/>
+   <origin xyz="0 0 0.087" rpy="0 0 0"/>
+</joint>
+<link name="chassis">
+   <visual>
+     <geometry>
+       <cylinder radius="0.17" length="0.14"/>
+     </geometry>
+     <origin xyz="0 0 0" rpy="0 0 0"/>
+     <material name="white"/>
+   </visual>
+   <collision>
+     <geometry>
+       <cylinder radius="0.17" length="0.14"/>
+     </geometry>
+     <origin xyz="0 0 0" rpy="0 0 0"/>
+   </collision>
+   <xacro:cylinder_inertia m="4" r="0.17" l="0.14" o_xyz="0 0 0" o_rpy="0 0 0" />
+</link>
+<link name="caster_wheel">
+   <visual>
+      <geometry>
+        <sphere radius="0.033"/>
+      </geometry>
+      <origin xyz="0 0 0" rpy="0 0 0"/>
+      <material name="gray"/>
+   </visual>
+   <collision>
+      <geometry>
+        <sphere radius="0.033"/>
+      </geometry>
+      <origin xyz="0 0 0" rpy="0 0 0"/>
+   </collision>
+   <xacro:sphere_inertia m="0.2" r="0.033" o_xyz="0 0 0" o_rpy="0 0 0" />
+</link>
+<joint name="caster_wheel_joint" type="fixed">
+    <parent link="chassis"/>
+    <child link="caster_wheel"/>
+    <origin xyz="0.12 0 -0.054" rpy="0 0 0"/>
+</joint>
+<joint name="left_wheel_joint" type="continuous">
+  <parent link="chassis"/>
+  <child link="left_wheel"/>
+  <origin xyz="0 0.115 -0.054" rpy="1.57 0 0" />
+  <axis xyz="0 0 -1"/>
+</joint>
+<link name="left_wheel">
+  <visual>
+      <geometry>
+          <cylinder radius="0.033" length="0.015"/>
+      </geometry>
+      <material name="gray"/>
+      <origin xyz="0 0 0" rpy="0 0 0" />
+  </visual>
+  <collision>
+    <geometry>
+        <cylinder radius="0.033" length="0.015"/>
+    </geometry>
+    <origin xyz="0 0 0" rpy="0 0 0" />
+</collision>
+<xacro:cylinder_inertia m="1" r="0.033" l="0.015" o_xyz="0 0 0" o_rpy="0 0 0" />
+</link>
+<joint name="right_wheel_joint" type="continuous">
+  <parent link="chassis"/>
+  <child link="right_wheel"/>
+  <origin xyz="0 -0.115 -0.054" rpy="1.57 0 0" />
+  <axis xyz="0 0 -1"/>
+</joint>
+<link name="right_wheel">
+  <visual>
+      <geometry>
+          <cylinder radius="0.033" length="0.015"/>
+      </geometry>
+      <material name="gray"/>
+      <origin xyz="0 0 0" rpy="0 0 0" />
+  </visual>
+  <collision>
+    <geometry>
+        <cylinder radius="0.033" length="0.015"/>
+    </geometry>
+    <origin xyz="0 0 0" rpy="0 0 0" />
+</collision>
+<xacro:cylinder_inertia m="1" r="0.033" l="0.015" o_xyz="0 0 0" o_rpy="0 0 0" />
+</link>
 </robot>
