Commit message: setup new frame

File: description/lidar.xacro (robot description, xacro)
@@ -7,5 +7,5 @@
         <parent link="chassis"/>
         <child link="laser_frame"/>
-        <origin xyz="0 0 0.06" rpy="0 0 0"/>
+        <origin xyz="0 0 0.115" rpy="0 0 0"/>
     </joint>
     <link name="laser_frame">

File: description/robot.urdf.xacro (robot description, xacro)
@@ -38,5 +38,5 @@
        <parent link="base_link"/>
        <child link="chassis"/>
-       <origin xyz="0 0 0.042" rpy="0 0 0"/>
+       <origin xyz="0 0 0.081" rpy="0 0 0"/>
    </joint>
    <link name="right_wheel">

Commit message: hdhdh

File: description/lidar.xacro (robot description, xacro)
@@ -5,5 +5,5 @@
    </material>
     <joint name="laser_joint" type="fixed">
-        <parent link="chassis"/>
+        <parent link="base_link"/>
         <child link="laser_frame"/>
         <origin xyz="0 0 0.095" rpy="0 0 0"/>

File: description/robot.urdf.xacro (robot description, xacro)
@@ -13,10 +13,10 @@
  <link name="base_footprint"/>
  <!-- Chassis link -->
- <joint name="chassis_joint" type="fixed">
+ <joint name="base_link_joint" type="fixed">
    <parent link="base_footprint"/>
-   <child link="chassis"/>
+   <child link="base_link"/>
    <origin xyz="0 0 0.087" rpy="0 0 0"/>
 </joint>
-<link name="chassis">
+<link name="base_link">
    <visual>
      <geometry>
@@ -51,10 +51,10 @@
 </link>
 <joint name="caster_wheel_joint" type="fixed">
-    <parent link="chassis"/>
+    <parent link="base_link"/>
     <child link="caster_wheel"/>
     <origin xyz="0.12 0 -0.054" rpy="0 0 0"/>
 </joint>
 <joint name="left_wheel_joint" type="continuous">
-  <parent link="chassis"/>
+  <parent link="base_link"/>
   <child link="left_wheel"/>
   <origin xyz="0 0.115 -0.054" rpy="1.57 0 0" />
@@ -78,5 +78,5 @@
 </link>
 <joint name="right_wheel_joint" type="continuous">
-  <parent link="chassis"/>
+  <parent link="base_link"/>
   <child link="right_wheel"/>
   <origin xyz="0 -0.115 -0.054" rpy="1.57 0 0" />

File: description/upbody.xacro (robot description, xacro)
@@ -8,5 +8,5 @@
    </material>
     <joint name="leftcol_joint" type="fixed">
-        <parent link="chassis"/>
+        <parent link="base_link"/>
         <child link="leftcol_frame"/>
         <origin xyz="0 0.165 0.12" rpy="0 0 0"/>
@@ -28,5 +28,5 @@
     </link>
     <joint name="rightcol_joint" type="fixed">
-        <parent link="chassis"/>
+        <parent link="base_link"/>
         <child link="rightcol_frame"/>
         <origin xyz="0 -0.165 0.12" rpy="0 0 0"/>
@@ -48,5 +48,5 @@
     </link>
     <joint name="backcol_joint" type="fixed">
-        <parent link="chassis"/>
+        <parent link="base_link"/>
         <child link="backcol_frame"/>
         <origin xyz="-0.165 0 0.12" rpy="0 0 0"/>
