Commit message: 5 commit

File: description/robot.urdf.xacro (robot description, xacro)
@@ -1,5 +1,5 @@
 <?xml version="1.0"?>
 <robot name="robot" xmlns:xacro="http://www.ros.org/wiki/xacro">
-  <xacro:include filename="common_properties.xacro" />
+  <xacro:include filename="inertial_macros.xacro" />
    <material name="white">
      <color rgba="1 1 1 1"/>
@@ -15,5 +15,5 @@
       <visual>
         <geometry>
-          <cylinder radius="0.1" length="0.124"/>
+          <cylinder radius="0.17" length="0.07"/>
         </geometry>
         <origin xyz="0 0 0" rpy="0 0 0"/>
@@ -22,14 +22,14 @@
       <collision>
         <geometry>
-          <cylinder radius="0.1" length="0.124"/>
+          <cylinder radius="0.17" length="0.07"/>
         </geometry>
         <origin xyz="0 0 0" rpy="0 0 0"/>
       </collision>
-      <xacro:cylinder_inertia m="1" r="0.1" l="0.124" o_xyz="0 0 0" o_rpy="0 0 0" />
+      <xacro:cylinder_inertia m="4" r="0.17" l="0.07" o_xyz="0 0 0" o_rpy="0 0 0" />
    </link>
    <joint name="base_joint" type="fixed">
        <parent link="base_footprint"/>
        <child link="base_link"/>
-       <origin xyz="0 0 0.079" rpy="0 0 0"/>
+       <origin xyz="0 0 0.035" rpy="0 0 0"/>
    </joint>
    <link name="raspberry_link">
@@ -52,10 +52,10 @@
       <parent link="base_link"/>
       <child link="raspberry_link"/>
-      <origin xyz="-0.06 0 0.0795" rpy="0 0 0"/>
+      <origin xyz="-0.10 0 0.07" rpy="0 0 0"/>
    </joint>
    <link name="right_wheel_link">
       <visual>
          <geometry>
-           <cylinder radius="0.033" length="0.03"/>
+           <cylinder radius="0.033" length="0.015"/>
          </geometry>
          <origin xyz="0 0 0" rpy="1.57 0 0"/>
@@ -64,14 +64,14 @@
       <collision>
          <geometry>
-           <cylinder radius="0.033" length="0.03"/>
+           <cylinder radius="0.033" length="0.015"/>
          </geometry>
          <origin xyz="0 0 0" rpy="1.57 0 0"/>
       </collision>
-      <xacro:cylinder_inertia m="0.1" r="0.033" l="0.03" o_xyz="0 0 0" o_rpy="1.57 0 0" />
+      <xacro:cylinder_inertia m="0.2" r="0.033" l="0.015" o_xyz="0 0 0" o_rpy="1.57 0 0" />
    </link>
    <joint name="base_right_wheel_joint" type="continuous">
       <parent link="base_link"/>
       <child link="right_wheel_link"/>
-      <origin xyz="0 -0.115 -0.045" rpy="0 0 0"/>
+      <origin xyz="0 -0.115 0" rpy="0 0 0"/>
       <axis xyz="0 1 0"/>
    </joint>
@@ -79,5 +79,5 @@
       <visual>
          <geometry>
-           <cylinder radius="0.033" length="0.03"/>
+           <cylinder radius="0.033" length="0.015"/>
          </geometry>
          <origin xyz="0 0 0" rpy="1.57 0 0"/>
@@ -86,14 +86,14 @@
       <collision>
          <geometry>
-           <cylinder radius="0.033" length="0.03"/>
+           <cylinder radius="0.033" length="0.015"/>
          </geometry>
          <origin xyz="0 0 0" rpy="1.57 0 0"/>
       </collision>
-      <xacro:cylinder_inertia m="0.1" r="0.033" l="0.03" o_xyz="0 0 0" o_rpy="1.57 0 0" />
+      <xacro:cylinder_inertia m="0.2" r="0.033" l="0.015" o_xyz="0 0 0" o_rpy="1.57 0 0" />
    </link>
    <joint name="base_left_wheel_joint" type="continuous">
       <parent link="base_link"/>
       <child link="left_wheel_link"/>
-      <origin xyz="0 0.115 -0.045" rpy="0 0 0"/>
+      <origin xyz="0 0.115 0" rpy="0 0 0"/>
       <axis xyz="0 1 0"/>
    </joint>

Commit message: sec

File: description/robot.urdf.xacro (robot description, xacro)
@@ -54,5 +54,5 @@
       <origin xyz="-0.10 0 0.0525" rpy="0 0 0"/>
    </joint>
-   <link name="right_wheel_link">
+   <link name="right_wheel">
       <visual>
          <geometry>
@@ -70,11 +70,11 @@
       <xacro:cylinder_inertia m="0.2" r="0.033" l="0.015" o_xyz="0 0 0" o_rpy="1.57 0 0" />
    </link>
-   <joint name="base_right_wheel_joint" type="continuous">
+   <joint name="right_wheel_joint" type="continuous">
       <parent link="base_link"/>
-      <child link="right_wheel_link"/>
+      <child link="right_wheel"/>
       <origin xyz="0 -0.115 -0.009" rpy="0 0 0"/>
       <axis xyz="0 1 0"/>
    </joint>
-   <link name="left_wheel_link">
+   <link name="left_wheel">
       <visual>
          <geometry>
@@ -92,11 +92,11 @@
       <xacro:cylinder_inertia m="0.2" r="0.033" l="0.015" o_xyz="0 0 0" o_rpy="1.57 0 0" />
    </link>
-   <joint name="base_left_wheel_joint" type="continuous">
+   <joint name="left_wheel_joint" type="continuous">
       <parent link="base_link"/>
-      <child link="left_wheel_link"/>
+      <child link="left_wheel"/>
       <origin xyz="0 0.115 -0.009" rpy="0 0 0"/>
       <axis xyz="0 1 0"/>
    </joint>
-   <link name="caster_wheel_link">
+   <link name="caster_wheel">
       <visual>
          <geometry>
@@ -114,7 +114,7 @@
       <xacro:sphere_inertia m="0.2" r="0.033" o_xyz="0 0 0" o_rpy="0 0 0" />
    </link>
-   <joint name="base_caster_wheel_joint" type="fixed">
+   <joint name="caster_wheel_joint" type="fixed">
        <parent link="base_link"/>
-       <child link="caster_wheel_link"/>
+       <child link="caster_wheel"/>
        <origin xyz="0.12 0 -0.009" rpy="0 0 0"/>
    </joint>

File: description/ros2_control.xacro (robot description, xacro)
@@ -4,6 +4,6 @@
             <hardware>
                 <plugin>diffdrive_arduino/DiffDriveArduino</plugin>
-                <param name="left_wheel_name">base_left_wheel_joint</param>
-                <param name="right_wheel_name">base_right_wheel_joint</param>
+                <param name="left_wheel_name">left_wheel_joint</param>
+                <param name="right_wheel_name">right_wheel_joint</param>
                 <param name="loop_rate">30</param>
                 <param name="device">/dev/ttyACM0</param>
@@ -12,5 +12,5 @@
                 <param name="enc_counts_per_rev">3430</param>
             </hardware>
-            <joint name="base_left_wheel_joint">
+            <joint name="left_wheel_joint">
                 <command_interface name="velocity">
                     <param name="min">-10</param>
@@ -20,5 +20,5 @@
                 <state_interface name="position"/>
             </joint>
-            <joint name="base_right_wheel_joint">
+            <joint name="right_wheel_joint">
                 <command_interface name="velocity">
                     <param name="min">-10</param>

Commit message: ros2_control work with humble

File: description/robot.urdf.xacro (robot description, xacro)
@@ -11,6 +11,12 @@
      <color rgba="0.5 0.5 0.5 1"/>
    </material>
+   <link name="base_link"/>
+   <joint name="base_footprint_joint" type="fixed">
+       <parent link="base_link"/>
+       <child link="base_footprint"/>
+       <origin xyz="0 0 0" rpy="0 0 0"/>
+   </joint>
    <link name="base_footprint"/>
-   <link name="base_link">
+   <link name="chassis">
       <visual>
         <geometry>
@@ -28,10 +34,10 @@
       <xacro:cylinder_inertia m="4" r="0.17" l="0.07" o_xyz="0 0 0" o_rpy="0 0 0" />
    </link>
-   <joint name="base_joint" type="fixed">
-       <parent link="base_footprint"/>
-       <child link="base_link"/>
+   <joint name="chassis_joint" type="fixed">
+       <parent link="base_link"/>
+       <child link="chassis"/>
        <origin xyz="0 0 0.042" rpy="0 0 0"/>
    </joint>
-   <link name="raspberry_link">
+   <link name="raspberry">
       <visual>
         <geometry>
@@ -49,7 +55,7 @@
       <xacro:box_inertia m="0.3" x="0.055" y="0.085" z="0.035" o_xyz="0 0 0" o_rpy="0 0 0" />
    </link>
-   <joint name="base_raspberry_joint" type="fixed">
-      <parent link="base_link"/>
-      <child link="raspberry_link"/>
+   <joint name="raspberry_joint" type="fixed">
+      <parent link="chassis"/>
+      <child link="raspberry"/>
       <origin xyz="-0.10 0 0.0525" rpy="0 0 0"/>
    </joint>
@@ -71,5 +77,5 @@
    </link>
    <joint name="right_wheel_joint" type="continuous">
-      <parent link="base_link"/>
+      <parent link="chassis"/>
       <child link="right_wheel"/>
       <origin xyz="0 -0.115 -0.009" rpy="0 0 0"/>
@@ -93,5 +99,5 @@
    </link>
    <joint name="left_wheel_joint" type="continuous">
-      <parent link="base_link"/>
+      <parent link="chassis"/>
       <child link="left_wheel"/>
       <origin xyz="0 0.115 -0.009" rpy="0 0 0"/>
@@ -115,5 +121,5 @@
    </link>
    <joint name="caster_wheel_joint" type="fixed">
-       <parent link="base_link"/>
+       <parent link="chassis"/>
        <child link="caster_wheel"/>
        <origin xyz="0.12 0 -0.009" rpy="0 0 0"/>

Commit message: add xbox 360 joystick

File: description/robot.urdf.xacro (robot description, xacro)
@@ -12,4 +12,11 @@
    </material>
    <link name="base_link"/>
+   <joint name="base_footprint_joint" type="fixed">
+        <parent link="base_link"/>
+        <child link="base_footprint"/>
+        <origin xyz="0 0 0" rpy="0 0 0"/>
+    </joint>
+    <link name="base_footprint">
+    </link>
    <link name="chassis">
       <visual>

Commit message: setup new frame

File: description/robot.urdf.xacro (robot description, xacro)
@@ -22,5 +22,5 @@
       <visual>
         <geometry>
-          <cylinder radius="0.17" length="0.07"/>
+          <cylinder radius="0.17" length="0.135"/>
         </geometry>
         <origin xyz="0 0 0" rpy="0 0 0"/>
@@ -29,9 +29,9 @@
       <collision>
         <geometry>
-          <cylinder radius="0.17" length="0.07"/>
+          <cylinder radius="0.17" length="0.135"/>
         </geometry>
         <origin xyz="0 0 0" rpy="0 0 0"/>
       </collision>
-      <xacro:cylinder_inertia m="4" r="0.17" l="0.07" o_xyz="0 0 0" o_rpy="0 0 0" />
+      <xacro:cylinder_inertia m="4" r="0.17" l="0.135" o_xyz="0 0 0" o_rpy="0 0 0" />
    </link>
    <joint name="chassis_joint" type="fixed">
@@ -39,25 +39,4 @@
        <child link="chassis"/>
        <origin xyz="0 0 0.042" rpy="0 0 0"/>
-   </joint>
-   <link name="raspberry">
-      <visual>
-        <geometry>
-          <box size="0.055 0.085 0.035"/>
-        </geometry>
-        <origin xyz="0 0 0" rpy="0 0 0"/>
-        <material name="green"/>
-      </visual>
-      <collision>
-        <geometry>
-          <box size="0.055 0.085 0.035"/>
-        </geometry>
-        <origin xyz="0 0 0" rpy="0 0 0"/>
-      </collision>
-      <xacro:box_inertia m="0.3" x="0.055" y="0.085" z="0.035" o_xyz="0 0 0" o_rpy="0 0 0" />
-   </link>
-   <joint name="raspberry_joint" type="fixed">
-      <parent link="chassis"/>
-      <child link="raspberry"/>
-      <origin xyz="-0.10 0 0.0525" rpy="0 0 0"/>
    </joint>
    <link name="right_wheel">

Commit message: js

File: description/robot.urdf.xacro (robot description, xacro)
@@ -59,5 +59,5 @@
       <parent link="chassis"/>
       <child link="right_wheel"/>
-      <origin xyz="0 -0.115 -0.009" rpy="0 0 0"/>
+      <origin xyz="0 -0.115 -0.017" rpy="0 0 0"/>
       <axis xyz="0 1 0"/>
    </joint>
@@ -81,5 +81,5 @@
       <parent link="chassis"/>
       <child link="left_wheel"/>
-      <origin xyz="0 0.115 -0.009" rpy="0 0 0"/>
+      <origin xyz="0 0.115 -0.017" rpy="0 0 0"/>
       <axis xyz="0 1 0"/>
    </joint>
@@ -103,5 +103,5 @@
        <parent link="chassis"/>
        <child link="caster_wheel"/>
-       <origin xyz="0.12 0 -0.009" rpy="0 0 0"/>
+       <origin xyz="0.12 0 -0.017" rpy="0 0 0"/>
    </joint>
 </robot>

Commit message: asdf

File: description/robot.urdf.xacro (robot description, xacro)
@@ -22,5 +22,5 @@
       <visual>
         <geometry>
-          <cylinder radius="0.17" length="0.135"/>
+          <cylinder radius="0.17" length="0.14"/>
         </geometry>
         <origin xyz="0 0 0" rpy="0 0 0"/>
@@ -29,14 +29,14 @@
       <collision>
         <geometry>
-          <cylinder radius="0.17" length="0.135"/>
+          <cylinder radius="0.17" length="0.14"/>
         </geometry>
         <origin xyz="0 0 0" rpy="0 0 0"/>
       </collision>
-      <xacro:cylinder_inertia m="4" r="0.17" l="0.135" o_xyz="0 0 0" o_rpy="0 0 0" />
+      <xacro:cylinder_inertia m="4" r="0.17" l="0.14" o_xyz="0 0 0" o_rpy="0 0 0" />
    </link>
    <joint name="chassis_joint" type="fixed">
        <parent link="base_link"/>
        <child link="chassis"/>
-       <origin xyz="0 0 0.081" rpy="0 0 0"/>
+       <origin xyz="0 0 0.07" rpy="0 0 0"/>
    </joint>
    <link name="right_wheel">

Commit message: jjs

File: description/robot.urdf.xacro (robot description, xacro)
@@ -12,10 +12,4 @@
   </material>
  <link name="base_footprint"/>
- <!-- Base link -->
- <joint name="base_link_joint" type="fixed">
-   <parent link="base_footprint"/>
-   <child link="base_link"/>
-   <origin xyz="0 0 0.087" rpy="0 0 0"/>
-</joint>
 <link name="base_link">
    <visual>
@@ -34,4 +28,10 @@
    <xacro:cylinder_inertia m="4" r="0.17" l="0.14" o_xyz="0 0 0" o_rpy="0 0 0" />
 </link>
+<!-- Base link -->
+ <joint name="base_link_joint" type="fixed">
+   <parent link="base_footprint"/>
+   <child link="base_link"/>
+   <origin xyz="0 0 0.087" rpy="0 0 0"/>
+</joint>
 <link name="caster_wheel">
    <visual>
@@ -55,4 +55,20 @@
     <origin xyz="0.12 0 -0.054" rpy="0 0 0"/>
 </joint>
+<link name="left_wheel">
+  <visual>
+      <geometry>
+          <cylinder radius="0.033" length="0.015"/>
+      </geometry>
+      <material name="gray"/>
+      <origin xyz="0 0 0" rpy="0 0 0" />
+  </visual>
+  <collision>
+    <geometry>
+        <cylinder radius="0.033" length="0.015"/>
+    </geometry>
+    <origin xyz="0 0 0" rpy="0 0 0" />
+</collision>
+<xacro:cylinder_inertia m="1" r="0.033" l="0.015" o_xyz="0 0 0" o_rpy="0 0 0" />
+</link>
 <joint name="left_wheel_joint" type="continuous">
   <parent link="base_link"/>
@@ -61,5 +77,5 @@
   <axis xyz="0 0 -1"/>
 </joint>
-<link name="left_wheel">
+<link name="right_wheel">
   <visual>
       <geometry>
@@ -83,19 +99,3 @@
   <axis xyz="0 0 -1"/>
 </joint>
-<link name="right_wheel">
-  <visual>
-      <geometry>
-          <cylinder radius="0.033" length="0.015"/>
-      </geometry>
-      <material name="gray"/>
-      <origin xyz="0 0 0" rpy="0 0 0" />
-  </visual>
-  <collision>
-    <geometry>
-        <cylinder radius="0.033" length="0.015"/>
-    </geometry>
-    <origin xyz="0 0 0" rpy="0 0 0" />
-</collision>
-<xacro:cylinder_inertia m="1" r="0.033" l="0.015" o_xyz="0 0 0" o_rpy="0 0 0" />
-</link>
 </robot>

File: description/upbody.xacro (robot description, xacro)
@@ -7,4 +7,19 @@
     <color rgba="1 1 1 1"/>
    </material>
+    <link name="leftcol_frame">
+        <visual>
+            <origin xyz="0 0 0"/>
+            <geometry>
+                <cylinder radius="0.005" length="0.10"/>
+            </geometry>
+            <material name="blac"/>
+        </visual>
+        <collision>
+            <geometry>
+                <cylinder radius="0.005" length="0.1"/>
+            </geometry>
+        </collision>
+        <xacro:cylinder_inertia m="1" r="0.005" l="0.1" o_xyz="0 0 0" o_rpy="0 0 0" />
+    </link>
     <joint name="leftcol_joint" type="fixed">
         <parent link="base_link"/>
@@ -12,5 +27,5 @@
         <origin xyz="0 0.165 0.12" rpy="0 0 0"/>
     </joint>
-    <link name="leftcol_frame">
+    <link name="rightcol_frame">
         <visual>
             <origin xyz="0 0 0"/>
@@ -32,5 +47,5 @@
         <origin xyz="0 -0.165 0.12" rpy="0 0 0"/>
     </joint>
-    <link name="rightcol_frame">
+    <link name="backcol_frame">
         <visual>
             <origin xyz="0 0 0"/>
@@ -52,24 +67,4 @@
         <origin xyz="-0.165 0 0.12" rpy="0 0 0"/>
     </joint>
-    <link name="backcol_frame">
-        <visual>
-            <origin xyz="0 0 0"/>
-            <geometry>
-                <cylinder radius="0.005" length="0.10"/>
-            </geometry>
-            <material name="blac"/>
-        </visual>
-        <collision>
-            <geometry>
-                <cylinder radius="0.005" length="0.1"/>
-            </geometry>
-        </collision>
-        <xacro:cylinder_inertia m="1" r="0.005" l="0.1" o_xyz="0 0 0" o_rpy="0 0 0" />
-    </link>
-    <joint name="body_joint" type="fixed">
-        <parent link="backcol_frame"/>
-        <child link="body_frame"/>
-        <origin xyz="0.165 0 0.23" rpy="0 0 0"/>
-    </joint>
     <link name="body_frame">
         <visual>
@@ -87,3 +82,8 @@
         <xacro:cylinder_inertia m="1" r="0.17" l="0.36" o_xyz="0 0 0" o_rpy="0 0 0" />
     </link>
+    <joint name="body_joint" type="fixed">
+        <parent link="backcol_frame"/>
+        <child link="body_frame"/>
+        <origin xyz="0.165 0 0.23" rpy="0 0 0"/>
+    </joint>
 </robot>
